File: PCB/FireKey.kicad_pcb (KiCad board)
At the start: 2 copper layers, 100 x 96.5 mm, 76 parts, among them SW1 SW_MEC_4A, U1 Arduino_Pro_Micro_USB-C

Commit message: worked on tracing pcb
Parts:
- H1, H2, H3, H4: moved to B.Cu
- turned H1 to 180 degrees
- turned H2 to 180 degrees
- turned H3 to 180 degrees
- turned H4 to 180 degrees
- turned R1 to 0 degrees
Routing:
- net VCC: track 54.2 -> 562.6 mm, vias 0 -> 7
- net Col2: track 0.00 -> 189.8 mm
- net Col1: track 0.00 -> 169.2 mm
- net Col0: track 0.00 -> 144.6 mm
- net Row4: track 38.1 -> 91.8 mm
- net SDA: track 0.00 -> 46.6 mm
- net LEDpin: track 0.00 -> 45.2 mm, vias 0 -> 1
- net SCL: track 0.00 -> 42.7 mm
- net Row3: track 38.1 -> 73.0 mm
- net Row0: track 38.1 -> 67.2 mm
- net Net-(LED3-Pad2): track 0.00 -> 27.2 mm
- net Net-(LED10-Pad4): track 0.00 -> 27.2 mm
- net Row2: track 38.1 -> 58.4 mm
- net Row1: track 38.1 -> 56.4 mm
- net Net-(LED8-Pad2): track 0.00 -> 14.1 mm
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
Commit message: worked on DRC errors
Parts:
- removed H1, H4: Pad, TestPoint:TestPoint_Pad_D2.5mm
- D1, D10, D11, D12, D13, D14, D15, D2, D3, D4, D5, D6, D7, D8, D9: footprint Diode_SMD:D_SOD-123 -> Custom_Parts:D_SOD-123
- moved H3 49.1 mm to (130.2, 113.9)
- moved H2 41.1 mm to (133.9, 113.8)
Routing:
- net Net-(LED6-Pad2): track 0.00 -> 26.7 mm, vias 0 -> 2
- net Net-(LED12-Pad2): track 0.00 -> 26.7 mm, vias 0 -> 2
- net VCC: track 562.6 -> 575.2 mm
- net GND: track 0.00 -> 7.08 mm
Other:
- board text added: "GND"
- board text added: "SDA SCL GND VCC"
- board text added: "VCC"
- board text added: "VCC GND SCL SDA"

Commit message: finished V0.0
Parts:
- added G***: LOGO, LOGO, F.Cu at (134.6, 91.4)
Other:
- board text added: "Czeschner Wolter 2022"
- board text added: "V0.0"

Commit message: fixed version number to V0.1
Other:
- board text added: "V0.1"
- board text removed: "V0.0"
Changed lines of the file:
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@@
     (title "FireKey PCB")
     (date "2022-11-29")
-    (rev "0.0")
+    (rev "0.1")
     (company "Daniel Czeschner & Frederik Wolter")
   )
@@
     (effects (font (size 1.6 1.6) (thickness 0.3)) (justify left mirror))
   )
-  (gr_text "V0.0" (at 141.605 143.51) (layer "B.SilkS")
+  (gr_text "V0.1" (at 141.605 143.51) (layer "B.SilkS")
     (effects (font (size 2 2) (thickness 0.4)) (justify mirror))
   )

Commit message: added Logo as footprint; worked on DRC
Parts:
- removed G***: LOGO, LOGO
- added G1: FireKey_Logo, Custom_Parts:FireKey_Logo, F.Cu at (134.6, 91.4)
