File: PCB_theory/FireKey_Theory.kicad_sch (KiCad schematic)
At the start: 0 parts

Commit message: Added button theory
Other:
- added sheet 1_Botton_Matrix (1_Botton_Matrix.kicad_sch)
- added sheet 1_Botton_Matrix_Complete (1_Botton_Matrix_Complete.kicad_sch)
- added sheet 1_Botton_Matrix_Diodes (1_Botton_Matrix_Diodes.kicad_sch)
- added sheet 1_Button_Single (1_Button_Single.kicad_sch)
