File: PCB_theory/1_Botton_Matrix_Complete.kicad_sch (KiCad schematic)
At the start: 30 parts

Commit message: minor changes to 1_botton_complete
Other:
- note removed: "DOWN-Key"
- note removed: "HOME-Key"
- note removed: "UP-Key"
Changed lines of the file:
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@@
     (stroke (width 0) (type default) (color 0 0 0 0))
-  )
-  (polyline (pts (xy 95.25 17.78) (xy 95.25 72.39))
-    (stroke (width 0) (type dot) (color 16 16 16 1))
   )
   (wire (pts (xy 80.01 38.1) (xy 97.79 38.1))
@@
     (stroke (width 0) (type default) (color 0 0 0 0))
   )
-  (text "HOME-Key" (at 110.49 49.53 0)
-    (effects (font (size 1.227 1.227)) (justify left bottom))
-  )
-  (text "UP-Key" (at 110.49 34.29 0)
-    (effects (font (size 1.27 1.27)) (justify left bottom))
-  )
-  (text "DOWN-Key" (at 110.49 64.77 0)
-    (effects (font (size 1.27 1.27)) (justify left bottom))
-  )
   (global_label "Col1" (shape input) (at 91.44 25.4 90) (fields_autoplaced)
